Commit message: refactor: consolidate RobotAPI and RobotConfigRegistry into unified RobotService
- Create unified RobotService consolidating robot discovery and config management
- Update RobotContext to use new service
- Update RobotManager with enhanced mesh path resolution
- Update URDFLoader to integrate with RobotService
- Update Controls component to use robotService
- Remove duplicate code (~200 lines eliminated)
- Improve error handling and fallback mechanisms
- Add unified logging and debugging capabilities

File: public/robots/techmanroboter/tm12/tm12.urdf (robot description, URDF)
Before this commit: robot tm12, 11 links, 10 joints
Links:
- link link_6: mass 0.65 -> 0.31; geometry collision mesh filename=package://tm_description/meshes/tm5-900/collision/tmr_iox_c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; visual mesh filename=package://tm_description/meshes/tm5-900/visual/tmr_iox.obj
Joints:
- joint shoulder_1_joint: limit lower=-4.71238898038469 upper=4.71238898038469 effort=353 velocity=2.0943951023931953 -> lower=-6.283185307179586 upper=6.283185307179586 effort=353 velocity=2.0943951023931953
- joint shoulder_2_joint: limit lower=-3.141592653589793 upper=3.141592653589793 effort=353 velocity=2.0943951023931953 -> lower=-6.283185307179586 upper=6.283185307179586 effort=353 velocity=2.0943951023931953
- joint wrist_1_joint: limit lower=-3.141592653589793 upper=3.141592653589793 effort=54 velocity=3.141592653589793 -> lower=-6.283185307179586 upper=6.283185307179586 effort=54 velocity=3.141592653589793
- joint wrist_2_joint: limit lower=-3.141592653589793 upper=3.141592653589793 effort=54 velocity=3.141592653589793 -> lower=-6.283185307179586 upper=6.283185307179586 effort=54 velocity=3.141592653589793
- joint wrist_3_joint: limit lower=-4.71238898038469 upper=4.71238898038469 effort=54 velocity=3.141592653589793 -> lower=-6.283185307179586 upper=6.283185307179586 effort=54 velocity=3.141592653589793
